File: Hardware/Edits/Eagle Files/buggym2017.brd (EAGLE design)
At the start: 88.9 x 81.3 mm, 6 parts, among them IC1 4001N, IC2 4075N, IC3 BCC, IC4 L293E

Commit message: Circuit Schematics
Finished circut schematics/layout, pending review on Wednesday 8/2
Parts:
- removed IC1: 4001N, 40xx:DIL14
- removed IC2: 4075N, 40xx:DIL14
- added IC1-NOR: 4001N, 40xx:DIL14
- added IC2-OR: 4075N, 40xx:DIL14
Connections:
- removed net N$1: IC1.3, IC2.2
- removed net N$4: IC1.4, IC2.4
- removed net VDD: IC1.14, IC2.14
- new net LINK_1: IC1-NOR.3, IC2-OR.2
- new net LINK_2: IC1-NOR.4, IC2-OR.4
- net 5V: now also IC1-NOR.14, IC2-OR.14
- net GND: now also IC1-NOR.7, IC2-OR.7; no longer IC1.7, IC2.7
- net LM: now also IC2-OR.9, IC4.7; no longer IC2.9
- net LO: now also IC1-NOR.6, IC2-OR.8
- net L_EYE: now also IC1-NOR.5, IC2-OR.1
- net RM: now also IC2-OR.6, IC4.10; no longer IC2.6
- net RO: now also IC1-NOR.2, IC2-OR.5
- net R_EYE: now also IC1-NOR.1, IC2-OR.3
Routing:
- net LO: track 0.00 -> 152.4 mm, vias 0 -> 8
- net RO: track 0.00 -> 121.9 mm, vias 0 -> 6
- net RM: track 0.00 -> 88.9 mm, vias 0 -> 4
- net L_EYE: track 0.00 -> 76.2 mm, vias 0 -> 4
- net R_EYE: track 0.00 -> 63.5 mm, vias 0 -> 4
- net 5V: track 109.2 -> 170.2 mm, vias 6 -> 14
- net LM: track 0.00 -> 53.3 mm, vias 0 -> 4
- net LINK_1: track 0.00 -> 22.9 mm, vias 0 -> 2
- net LINK_2: track 0.00 -> 20.3 mm
- net GND: track 159.9 -> 165.1 mm

Commit message: Week 4 Hardware
Circuit Layouts and Schematics - FINAL
Parts:
- moved IC2-OR 7.62 mm to (82.5, 15.2)
- moved IC1-NOR 5.08 mm to (49.5, 15.2)
Routing:
- net LINK_1: track 22.9 -> 86.4 mm, vias 2 -> 6
- net LINK_2: track 20.3 -> 63.5 mm, vias 0 -> 6
- net GND: track 165.1 -> 203.2 mm
- net LO: track 152.4 -> 175.3 mm
- net RO: track 121.9 -> 142.2 mm
- net R_EYE: track 63.5 -> 73.7 mm
- net L_EYE: track 76.2 -> 86.4 mm
- net 5V: track 170.2 -> 177.8 mm
- net RM: track 88.9 -> 96.5 mm
- net LM: track 53.3 -> 50.8 mm
Other:
- board text added: "X"
